Commit message: after cloning navigation package

File: diff_robot/urdf/diff_robot.urdf (robot description, URDF)
Before this commit: robot diff_robot, 7 links, 6 joints
Links:
- link base_link: geometry visual box size=0.7 0.4 0.2
Joints:
- joint base_lidar_joint: origin xyz=0.0 0.0 0.20 rpy=0.0 0.0 0.0 -> xyz=0.0 0.0 0.225 rpy=0.0 0.0 0.0
- joint left_wheel_joint: origin xyz=0.0 0.3 0.0 rpy=0 0.0 0.0 -> xyz=-0.175 0.225 0.0 rpy=0 0.0 0.0
- joint right_wheel_joint: origin xyz=0.0 -0.3 0.0 rpy=0 0.0 0.0 -> xyz=-0.175 -0.225 0.0 rpy=0 0.0 0.0

File: diff_robot/urdf/robomuse.urdf (robot description, URDF)
Before this commit: robot diff_robot, 7 links, 6 joints
Links:
- removed link caster_wheel
- removed link lidar_link
- added link caster_wheel1, mass 0.1; collision sphere radius=0.05; visual sphere radius=0.05
- added link caster_wheel2, mass 0.1; collision sphere radius=0.05; visual sphere radius=0.05
- added link caster_wheel3, mass 0.1; collision sphere radius=0.05; visual sphere radius=0.05
- added link caster_wheel4, mass 0.1; collision sphere radius=0.05; visual sphere radius=0.05
- added link lidar, mass 0.114; collision cylinder length=0.05 radius=0.05; visual cylinder length=0.05 radius=0.1
- link left_wheel: geometry collision cylinder length=0.05 radius=0.0625; visual cylinder length=0.05 radius=0.0625
- link right_wheel: geometry collision cylinder length=0.05 radius=0.0625; visual cylinder length=0.05 radius=0.0625
Joints:
- removed joint caster_wheel_joint
- added joint caster_wheel_joint_Back_left: type fixed, parent base_link, child caster_wheel4, origin xyz=-0.35 0.2 -0.05 rpy=0.0 0.0 0.0
- added joint caster_wheel_joint_Back_right: type fixed, parent base_link, child caster_wheel3, origin xyz=-0.35 -0.2 -0.05 rpy=0.0 0.0 0.0
- added joint caster_wheel_joint_Front_left: type fixed, parent base_link, child caster_wheel2, origin xyz=0.35 -0.2 -0.05 rpy=0.0 0.0 0.0
- added joint caster_wheel_joint_Front_right: type fixed, parent base_link, child caster_wheel1, origin xyz=0.35 0.2 -0.05 rpy=0.0 0.0 0.0
- joint base_lidar_joint: child lidar_link -> lidar
- joint left_wheel_joint: axis 0.0 1.0 0.0 -> (none); limit effort=100 velocity=1.0 -> (none); origin xyz=0.0 0.3 0.0 rpy=0 0.0 0.0 -> xyz=0.0 0.270 0.0 rpy=0 0 0; type continuous -> fixed
- joint right_wheel_joint: axis 0.0 1.0 0.0 -> (none); limit effort=100 velocity=1.0 -> (none); origin xyz=0.0 -0.3 0.0 rpy=0 0.0 0.0 -> xyz=0.0 -0.270 0.0 rpy=0 0 0; type continuous -> fixed
