Commit message: gazebo and real robot lauches usb renaming

File: diff_robot/urdf/robomuse.urdf (robot description, URDF)
Before this commit: robot diff_robot, 10 links, 9 joints
Links:
- link left_wheel: geometry collision cylinder length=0.05 radius=0.10625; visual cylinder length=0.05 radius=0.10625
- link right_wheel: geometry collision cylinder length=0.05 radius=0.10625; visual cylinder length=0.05 radius=0.10625
Joints:
- joint left_wheel_joint: axis (none) -> 0 1 0; limit (none) -> effort=10 velocity=10
- joint right_wheel_joint: axis (none) -> 0 1 0; limit (none) -> effort=10 velocity=10
